Commit message: Update gripper config

File: abb_irb1200_support/urdf/irb1200_7_70_macro.xacro (robot description, xacro)
@@ -184,5 +184,5 @@
     <joint name="${prefix}flange-tool0" type="fixed">
       <!-- <origin xyz="0 -0.18 0" rpy="${radians(90)} 0 0" /> -->
-      <origin xyz="0.188 0 0" rpy="0 0 0" />
+      <origin xyz="0.126 0 0" rpy="0 0 0" />
       <parent link="${prefix}flange" />
       <child link="${prefix}tool0" />

Commit message: Add 3 more gripper configurations

File: abb_irb1200_support/urdf/irb1200_7_70_macro.xacro (robot description, xacro)
@@ -161,10 +161,16 @@
       <collision name="collision">
         <geometry>
-          <mesh filename="package://abb_irb1200_support/meshes/vacuum_gripper_vgc10/irb1200_7_70_vacuum_gripper_vgc10_b.stl" />
+          <mesh filename="package://abb_irb1200_support/meshes/vacuum_gripper_vgc10/irb1200_7_70_vacuum_gripper_vgc10_15mm.stl" />
+          <!-- <mesh filename="package://abb_irb1200_support/meshes/vacuum_gripper_vgc10/irb1200_7_70_vacuum_gripper_vgc10_30mm.stl" /> -->
+          <!-- <mesh filename="package://abb_irb1200_support/meshes/vacuum_gripper_vgc10/irb1200_7_70_vacuum_gripper_vgc10_40mm_short.stl" /> -->
+          <!-- <mesh filename="package://abb_irb1200_support/meshes/vacuum_gripper_vgc10/irb1200_7_70_vacuum_gripper_vgc10_40mm_long.stl" /> -->
         </geometry>
       </collision>
       <visual name="visual">
         <geometry>
-          <mesh filename="package://abb_irb1200_support/meshes/vacuum_gripper_vgc10/irb1200_7_70_vacuum_gripper_vgc10_b.stl" />
+          <mesh filename="package://abb_irb1200_support/meshes/vacuum_gripper_vgc10/irb1200_7_70_vacuum_gripper_vgc10_15mm.stl" />
+          <!-- <mesh filename="package://abb_irb1200_support/meshes/vacuum_gripper_vgc10/irb1200_7_70_vacuum_gripper_vgc10_30mm.stl" /> -->
+          <!-- <mesh filename="package://abb_irb1200_support/meshes/vacuum_gripper_vgc10/irb1200_7_70_vacuum_gripper_vgc10_40mm_short.stl" /> -->
+          <!-- <mesh filename="package://abb_irb1200_support/meshes/vacuum_gripper_vgc10/irb1200_7_70_vacuum_gripper_vgc10_40mm_long.stl" /> -->
         </geometry>
         <material
